File: Carrier-Board.sch (KiCad schematic (older format))
At the start: 45 parts, among them J1 CONN_3-6318491-6, J10 Conn_02x03_Odd_Even, J2 Conn_01x0, J3 Conn_02x26_Odd_Even, J4 SI-51009-F, J5 Conn_02x26_Odd_Even, J6 Conn_01x03_Male, J7 Conn_01x03_Male, J8 Conn_01x06_Male, J9 Conn_02x04_Odd_Even, SW1 SW_Push, SW2 SW_Push, SW3 SW_Push, U1 MPM3620, U2 MPM3620, U9 MSATA-Socket

Commit message: lib stuff'
Parts:
- D5: symbol BusSimulator-cache:D_Zener -> Carrier-Board-rescue:D_Zener-BusSimulator-cache
- D6, D7, D8: symbol BusSimulator-cache:LED -> Carrier-Board-rescue:LED-BusSimulator-cache
- R1, R10, R11, R12, R13, R2, R23, R24, R25, R3, R32, R4, R5, R6, R7, R8, R9: symbol BusSimulator-cache:R -> Carrier-Board-rescue:R-BusSimulator-cache
Changed lines of the file:
@@
 EESchema Schematic File Version 4
+LIBS:Carrier-Board-cache
 EELAYER 26 0
 EELAYER END
@@
 $EndComp
 $Comp
-L BusSimulator-cache:GNDREF #PWR01
+L Carrier-Board-rescue:GNDREF-BusSimulator-cache #PWR01
 U 1 1 59F6A60F
 P 2325 1575
@@
 $EndComp
 $Comp
-L BusSimulator-cache:R R1
+L Carrier-Board-rescue:R-BusSimulator-cache R1
 U 1 1 59F6ABD8
 P 3150 3550
@@
 $EndComp
 $Comp
-L BusSimulator-cache:R R2
+L Carrier-Board-rescue:R-BusSimulator-cache R2
 U 1 1 59F6ACFA
 P 3150 3850
@@
 $EndComp
 $Comp
-L BusSimulator-cache:GNDA #PWR02
+L Carrier-Board-rescue:GNDA-BusSimulator-cache #PWR02
 U 1 1 59F6AEAC
 P 3150 4000
@@
 $EndComp
 $Comp
-L BusSimulator-cache:R R3
+L Carrier-Board-rescue:R-BusSimulator-cache R3
 U 1 1 59F6AF4C
 P 2650 1500
@@
 $EndComp
 $Comp
-L BusSimulator-cache:GNDA #PWR03
+L Carrier-Board-rescue:GNDA-BusSimulator-cache #PWR03
 U 1 1 59F6AF94
 P 1800 3250
@@
 $EndComp
 $Comp
-L BusSimulator-cache:R R4
+L Carrier-Board-rescue:R-BusSimulator-cache R4
 U 1 1 59FA907E
 P 3075 1950
@@
 $EndComp
 $Comp
-L BusSimulator-cache:GNDA #PWR04
+L Carrier-Board-rescue:GNDA-BusSimulator-cache #PWR04
 U 1 1 59FA90DC
 P 3300 2000
@@
 $EndComp
 $Comp
-L BusSimulator-cache:+5V #PWR05
+L Carrier-Board-rescue:+5V-BusSimulator-cache #PWR05
 U 1 1 59FAA2C5
 P 3150 2800
@@
 $EndComp
 $Comp
-L BusSimulator-cache:GNDREF #PWR06
+L Carrier-Board-rescue:GNDREF-BusSimulator-cache #PWR06
 U 1 1 59FAACBA
 P 2275 4575
@@
 $EndComp
 $Comp
-L BusSimulator-cache:R R5
+L Carrier-Board-rescue:R-BusSimulator-cache R5
 U 1 1 59FAACC0
 P 3100 6550
@@
 $EndComp
 $Comp
-L BusSimulator-cache:R R6
+L Carrier-Board-rescue:R-BusSimulator-cache R6
 U 1 1 59FAACC6
 P 3100 6850
@@
 $EndComp
 $Comp
-L BusSimulator-cache:GNDA #PWR07
+L Carrier-Board-rescue:GNDA-BusSimulator-cache #PWR07
 U 1 1 59FAACCC
 P 3100 7000
@@
 $EndComp
 $Comp
-L BusSimulator-cache:R R7
+L Carrier-Board-rescue:R-BusSimulator-cache R7
 U 1 1 59FAACD2
 P 2600 4500
@@
 $EndComp
 $Comp
-L BusSimulator-cache:GNDA #PWR08
+L Carrier-Board-rescue:GNDA-BusSimulator-cache #PWR08
 U 1 1 59FAACD8
 P 1750 6250
@@
 $EndComp
 $Comp
-L BusSimulator-cache:R R8
+L Carrier-Board-rescue:R-BusSimulator-cache R8
 U 1 1 59FAACF4
 P 3025 4950
@@
 $EndComp
 $Comp
-L BusSimulator-cache:GNDA #PWR09
+L Carrier-Board-rescue:GNDA-BusSimulator-cache #PWR09
 U 1 1 59FAACFB
 P 3250 5000
@@
 $EndComp
 $Comp
-L BusSimulator-cache:+3.3V #PWR010
+L Carrier-Board-rescue:+3.3V-BusSimulator-cache #PWR010
 U 1 1 59FAAF36
 P 3100 5800
@@
 PCE3900CT-ND
 $Comp
-L BusSimulator-cache:GNDREF #PWR011
+L Carrier-Board-rescue:GNDREF-BusSimulator-cache #PWR011
 U 1 1 59FACA7B
 P 3450 2550
@@
 $EndComp
 $Comp
-L BusSimulator-cache:GNDREF #PWR012
+L Carrier-Board-rescue:GNDREF-BusSimulator-cache #PWR012
 U 1 1 59FACBAF
 P 3500 5500
@@
 $EndComp
 $Comp
-L BusSimulator-cache:GNDREF #PWR013
+L Carrier-Board-rescue:GNDREF-BusSimulator-cache #PWR013
 U 1 1 59FACE9C
 P 3000 3550
@@
 $EndComp
 $Comp
-L BusSimulator-cache:GNDREF #PWR014
+L Carrier-Board-rescue:GNDREF-BusSimulator-cache #PWR014
 U 1 1 59FAD007
 P 2250 1250
@@
 $EndComp
 $Comp
-L BusSimulator-cache:GNDREF #PWR015
+L Carrier-Board-rescue:GNDREF-BusSimulator-cache #PWR015
 U 1 1 59FB82F0
 P 2250 4200
@@
 $EndComp
 $Comp
-L BusSimulator-cache:GNDREF #PWR016
+L Carrier-Board-rescue:GNDREF-BusSimulator-cache #PWR016
 U 1 1 59FB843A
 P 2950 6550
@@
 mCOM_GND
 $Comp
-L BusSimulator-cache:+12V #PWR017
+L Carrier-Board-rescue:+12V-BusSimulator-cache #PWR017
 U 1 1 5A040DA3
 P 2500 1500
@@
 $EndComp
 $Comp
-L BusSimulator-cache:+12V #PWR018
+L Carrier-Board-rescue:+12V-BusSimulator-cache #PWR018
 U 1 1 5A040EAE
 P 2450 4500
@@
 $EndComp
 $Comp
-L BusSimulator-cache:+12V #PWR019
+L Carrier-Board-rescue:+12V-BusSimulator-cache #PWR019
 U 1 1 5A0413FE
 P 1250 1850
@@
 $EndComp
 $Comp
-L BusSimulator-cache:GNDREF #PWR020
+L Carrier-Board-rescue:GNDREF-BusSimulator-cache #PWR020
 U 1 1 5A04143A
 P 900 1750
@@
 Break out\n
 $Comp
-L BusSimulator-cache:LED D7
+L Carrier-Board-rescue:LED-BusSimulator-cache D7
 U 1 1 5A07DE5B
 P 6350 1500
@@
 LED Indicators\n
 $Comp
-L BusSimulator-cache:LED D6
+L Carrier-Board-rescue:LED-BusSimulator-cache D6
 U 1 1 5A08439E
 P 6350 1800
@@
 $EndComp
 $Comp
-L BusSimulator-cache:LED D8
+L Carrier-Board-rescue:LED-BusSimulator-cache D8
 U 1 1 5A084441
 P 6350 2100
@@
 mCOM_5V_SBY
 $Comp
-L BusSimulator-cache:R R23
+L Carrier-Board-rescue:R-BusSimulator-cache R23
 U 1 1 5A0890AC
 P 6650 1500
@@
 $EndComp
 $Comp
-L BusSimulator-cache:R R24
+L Carrier-Board-rescue:R-BusSimulator-cache R24
 U 1 1 5A0891D7
 P 6650 1800
@@
 $EndComp
 $Comp
-L BusSimulator-cache:R R25
+L Carrier-Board-rescue:R-BusSimulator-cache R25
 U 1 1 5A0892AA
 P 6650 2100
@@
 $EndComp
 $Comp
-L BusSimulator-cache:GNDREF #PWR021
+L Carrier-Board-rescue:GNDREF-BusSimulator-cache #PWR021
 U 1 1 5A08977E
 P 7000 2500
@@
 Spring 2018\n\n
 $Comp
-L BusSimulator-cache:D_Zener D5
+L Carrier-Board-rescue:D_Zener-BusSimulator-cache D5
 U 1 1 5A07A33B
 P 6050 1800
@@
 +3.3V
 $Comp
-L BusSimulator-cache:GNDREF #PWR022
+L Carrier-Board-rescue:GNDREF-BusSimulator-cache #PWR022
 U 1 1 5A0C1B77
 P 3700 8250
@@
 $EndComp
 $Comp
-L BusSimulator-cache:GNDREF #PWR023
+L Carrier-Board-rescue:GNDREF-BusSimulator-cache #PWR023
 U 1 1 5A0C1C29
 P 3900 10650
@@
 $EndComp
 $Comp
-L BusSimulator-cache:GNDREF #PWR024
+L Carrier-Board-rescue:GNDREF-BusSimulator-cache #PWR024
 U 1 1 5A0C1CDB
 P 4000 9450
@@
 $EndComp
 $Comp
-L BusSimulator-cache:GNDREF #PWR025
+L Carrier-Board-rescue:GNDREF-BusSimulator-cache #PWR025
 U 1 1 5A0C1D8D
 P 4000 9050
@@
 $EndComp
 $Comp
-L BusSimulator-cache:GNDREF #PWR026
+L Carrier-Board-rescue:GNDREF-BusSimulator-cache #PWR026
 U 1 1 5A0C1E3F
 P 4000 8750
@@
 $EndComp
 $Comp
-L BusSimulator-cache:GNDREF #PWR027
+L Carrier-Board-rescue:GNDREF-BusSimulator-cache #PWR027
 U 1 1 5A0C1EF1
 P 4000 9850
@@
 SATA0_RX-
 $Comp
-L BusSimulator-cache:GNDREF #PWR028
+L Carrier-Board-rescue:GNDREF-BusSimulator-cache #PWR028
 U 1 1 5A0C49FB
 P 1800 10400
@@
 $EndComp
 $Comp
-L BusSimulator-cache:GNDREF #PWR029
+L Carrier-Board-rescue:GNDREF-BusSimulator-cache #PWR029
 U 1 1 5A0C4BAB
 P 1900 10050
@@
 Sata Connector\n
 $Comp
-L BusSimulator-cache:GNDREF #PWR030
+L Carrier-Board-rescue:GNDREF-BusSimulator-cache #PWR030
 U 1 1 5A0C6A3D
 P 1450 8950
@@
 $EndComp
 $Comp
-L BusSimulator-cache:GNDREF #PWR031
+L Carrier-Board-rescue:GNDREF-BusSimulator-cache #PWR031
 U 1 1 5A0C6D48
 P 1500 9350
@@
 $EndComp
 $Comp
-L BusSimulator-cache:R R32
+L Carrier-Board-rescue:R-BusSimulator-cache R32
 U 1 1 5A0C7549
 P 1600 8300
@@
 $EndComp
 $Comp
-L BusSimulator-cache:GNDREF #PWR032
+L Carrier-Board-rescue:GNDREF-BusSimulator-cache #PWR032
 U 1 1 5A0C77C7
 P 1600 8450
@@
 $EndComp
 $Comp
-L BusSimulator-cache:GNDREF #PWR033
+L Carrier-Board-rescue:GNDREF-BusSimulator-cache #PWR033
 U 1 1 5A0DCFAA
 P 750 8350
@@
 $EndComp
 $Comp
-L BusSimulator-cache:GNDREF #PWR034
+L Carrier-Board-rescue:GNDREF-BusSimulator-cache #PWR034
 U 1 1 5A0DD07C
 P 1100 9050
@@
 $EndComp
 $Comp
-L BusSimulator-cache:GNDREF #PWR035
+L Carrier-Board-rescue:GNDREF-BusSimulator-cache #PWR035
 U 1 1 5A0DDC34
 P 4500 8450
@@
 $EndComp
 $Comp
-L BusSimulator-cache:GNDREF #PWR036
+L Carrier-Board-rescue:GNDREF-BusSimulator-cache #PWR036
 U 1 1 5A0B68CF
 P 8750 1600
@@
 GBE0_CTREF(GND)
 $Comp
-L BusSimulator-cache:GNDREF #PWR037
+L Carrier-Board-rescue:GNDREF-BusSimulator-cache #PWR037
 U 1 1 5A6D828B
 P 6150 5750
@@
 $EndComp
 $Comp
-L BusSimulator-cache:R R9
+L Carrier-Board-rescue:R-BusSimulator-cache R9
 U 1 1 5A6D8633
 P 5700 5600
@@
 $EndComp
 $Comp
-L BusSimulator-cache:R R10
+L Carrier-Board-rescue:R-BusSimulator-cache R10
 U 1 1 5A6D9C5A
 P 6650 5350
@@
 $EndComp
 $Comp
-L BusSimulator-cache:GNDREF #PWR038
+L Carrier-Board-rescue:GNDREF-BusSimulator-cache #PWR038
 U 1 1 5A6D9E6B
 P 7250 5450
@@
 $EndComp
 $Comp
-L BusSimulator-cache:GNDREF #PWR039
+L Carrier-Board-rescue:GNDREF-BusSimulator-cache #PWR039
 U 1 1 5A6DAA22
 P 7300 5050
@@
 $EndComp
 $Comp
-L BusSimulator-cache:GNDREF #PWR040
+L Carrier-Board-rescue:GNDREF-BusSimulator-cache #PWR040
 U 1 1 5A6DB372
 P 5150 4750
@@
 WAKE1n
 $Comp
-L BusSimulator-cache:R R11
+L Carrier-Board-rescue:R-BusSimulator-cache R11
 U 1 1 5A6E9EDA
 P 14550 850
@@
 $EndComp
 $Comp
-L BusSimulator-cache:R R12
+L Carrier-Board-rescue:R-BusSimulator-cache R12
 U 1 1 5A6EA119
 P 14650 1600
@@
 $EndComp
 $Comp
-L BusSimulator-cache:R R13
+L Carrier-Board-rescue:R-BusSimulator-cache R13
 U 1 1 5A6EA1A0
 P 14650 2450
@@
 Connection ~ 14400 2450
 $Comp
-L BusSimulator-cache:GNDREF #PWR041
+L Carrier-Board-rescue:GNDREF-BusSimulator-cache #PWR041
 U 1 1 5A6EC603
 P 14350 1300
@@
 $EndComp
 $Comp
-L BusSimulator-cache:GNDREF #PWR042
+L Carrier-Board-rescue:GNDREF-BusSimulator-cache #PWR042
 U 1 1 5A6EC92F
 P 14400 2100
@@
 $EndComp
 $Comp
-L BusSimulator-cache:GNDREF #PWR043
+L Carrier-Board-rescue:GNDREF-BusSimulator-cache #PWR043
 U 1 1 5A6ECB43
 P 14400 3000
