File: Carrier-Board.sch (KiCad schematic (older format))
At the start: 56 parts, among them J1 CONN_3-6318491-6, J10 Conn_02x03_Odd_Even, J2 Conn_01x0, J3 Conn_02x26_Odd_Even, J4 SI-51009-F, J5 Conn_02x26_Odd_Even, J6 Conn_01x03_Male, J7 Conn_01x03_Male, J8 Conn_01x06_Male, J9 Conn_02x04_Odd_Even, SW1 SW_Push, SW2 SW_Push, SW3 SW_Push, U1 MPM3620, U2 MPM3620, U9 MSATA-Socket

Commit message: added usb
Parts:
- removed C? (x2): 100nF, symbol Device:C
- removed C?: 4.7nF, symbol Device:C
- removed C?: 10nF, symbol Device:C
- removed C? (x2): 47pF, symbol Device:C
- removed L?: Ferrite_Bead, symbol Device:Ferrite_Bead
- removed R? (x2): 27R, symbol Device:R
- removed U?: FT230X, symbol RS232_FTDI:FT230X
- added C? (x2): .1uF, Capacitors_SMD:C_0603, symbol Device:C
- added C?: 4.7uF, Capacitors_SMD:C_0603, symbol Device:C
- added D?: PESD12VL2BT,215, Diodes_SMD:D_SOT-23_NKA, symbol Power_Protection:SP0502BAJT
- added R?: 4.7K, Resistors_SMD:R_0603, symbol BusSimulator-rescue:R
- added R?: 10K, Resistors_SMD:R_0603, symbol BusSimulator-rescue:R
- added U?: MAX3221, symbol Interface_UART:MAX3221
- added U?: FT232RQ, FT232RQ:QFN50P500X500X100-33N, symbol FT232RQ:FT232RQ
- J?: footprint (none) -> Connectors_USB:USB_Micro-B_Molex-105017-0001
Connections:
- net labels added: Reset#
- wire segments 178 -> 170
- no-connect marks 0 -> 15
Other:
- moved on the sheet: R10, R9

Commit message: Finished Schematic for RS232 to USB
Parts:
- removed J4: SI-51009-F, Carrier-Board:SI-51009-F, symbol Connector_Generic:Conn_02x09_Odd_Even
- removed R10, R9: 330, Resistors_SMD:R_0805, symbol Carrier-Board-rescue:R-BusSimulator-cache
- added C?: 47nF, Capacitors_SMD:C_0603, symbol Device:C
- added C? (x3): .33uF, Capacitors_SMD:C_0603, symbol Device:C
- added C?: .1uF, Capacitors_SMD:C_0603, symbol Device:C
- added D? (x2): LED, Diodes_SMD:D_0805, symbol BusSimulator-rescue:LED
- added J?: SI-51009-F, Carrier-Board:SI-51009-F, symbol Connector_Generic:Conn_02x09_Odd_Even
- added R? (x2): 200, Resistors_SMD:R_0603, symbol BusSimulator-rescue:R
- added R?: 10K, Resistors_SMD:R_0603, symbol BusSimulator-rescue:R
- added R? (x2): 330, Resistors_SMD:R_0805, symbol Carrier-Board-rescue:R-BusSimulator-cache
- U?: footprint (none) -> Housings_SSOP:SSOP-16_5.3x6.2mm_Pitch0.65mm
Connections:
- net labels added: RXD, TXD
- wire segments 170 -> 206
- no-connect marks 15 -> 18
Other:
- note added: "USB to RS232\n"
- note added: "polarized +\n"
- note added: "polarized -\n\n"
- moved on the sheet: D5, D6, D7, D8, R23, R24, R25

Commit message: ---
Parts:
- J7: footprint Pin_Headers:Pin_Header_Angled_1x03_Pitch2.54mm -> TestPoint:TestPoint_Pad_D3.0mm
- gave numbers to parts that had none: 22
