File: Carrier-Board.sch (KiCad schematic (older format))
At the start: 64 parts, among them J1 CONN_3-6318491-6, J10 Conn_02x03_Odd_Even, J11 USB_B_Micro, J2 Conn_01x0, J3 Conn_02x26_Odd_Even, J4 SI-51009-F, J5 Conn_02x26_Odd_Even, J6 Conn_01x03_Male, J7 Conn_01x03_Male, J8 Conn_01x06_Male, J9 Conn_02x04_Odd_Even, SW1 SW_Push, SW2 SW_Push, SW3 SW_Push, U1 MPM3620, U2 MPM3620, U3 MAX3221, U4 FT232RQ, U9 MSATA-Socket

Commit message: Change footprint sizes
Parts:
- C1, C2, C3: footprint Capacitors_SMD:C_0805 -> Capacitor_SMD:C_0805_2012Metric
- C10, C11, C12, C27, C28, C29, C5, C6, C7, C8, C9: footprint Capacitors_SMD:C_0603 -> Capacitor_SMD:C_0603_1608Metric
- C4: footprint Capacitors_SMD:C_0805 -> Capacitor_SMD:C_0603_1608Metric
- D2, D3: footprint Diodes_SMD:D_0805 -> Diode_SMD:D_0805_2012Metric
- D6, D7, D8: footprint Diodes_SMD:D_1206 -> Diode_SMD:D_0805_2012Metric
- G1: footprint BusSimulator:LetSatLogo440 -> Carrier-Board:LetSat_Logo_440
- J1: footprint BusSimulator:ComExpressMini10 -> Carrier-Board:ComExpressMini10
- R1, R16, R2, R3, R32, R4, R5, R6, R7, R8, R9: footprint Resistors_SMD:R_0805 -> Resistor_SMD:R_0603_1608Metric
- R10, R11, R12, R13, R14, R15, R17, R18, R23, R24, R25: footprint Resistors_SMD:R_0603 -> Resistor_SMD:R_0603_1608Metric
- U1, U2: footprint BusSimulator:QFN-20 -> Carrier-Board:QFN-20
Connections:
- wire segments 206 -> 209

Commit message: Added 3d models
Parts:
- D2, D3: symbol BusSimulator-rescue:LED -> Carrier-Board-rescue:LED-BusSimulator-rescue
- R10, R14, R15, R17, R18: symbol BusSimulator-rescue:R -> Carrier-Board-rescue:R-BusSimulator-rescue
Changed lines of the file:
@@
 Connection ~ 7450 10800
 $Comp
-L BusSimulator-rescue:R R15
+L Carrier-Board-rescue:R-BusSimulator-rescue R15
 U 1 1 5BB25F1C
 P 6300 10250
@@
 Reset#
 $Comp
-L BusSimulator-rescue:R R10
+L Carrier-Board-rescue:R-BusSimulator-rescue R10
 U 1 1 5BB3EBD3
 P 6000 10250
@@
 	7950 7950 7950 7000
 $Comp
-L BusSimulator-rescue:LED D3
+L Carrier-Board-rescue:LED-BusSimulator-rescue D3
 U 1 1 5BABB0D8
 P 7950 6500
@@
 $EndComp
 $Comp
-L BusSimulator-rescue:LED D2
+L Carrier-Board-rescue:LED-BusSimulator-rescue D2
 U 1 1 5BAD1E5C
 P 7750 6500
@@
 $EndComp
 $Comp
-L BusSimulator-rescue:R R17
+L Carrier-Board-rescue:R-BusSimulator-rescue R17
 U 1 1 5BAD9A4D
 P 7750 6850
@@
 $EndComp
 $Comp
-L BusSimulator-rescue:R R18
+L Carrier-Board-rescue:R-BusSimulator-rescue R18
 U 1 1 5BAD9B89
 P 7950 6850
@@
 	6900 4500 7300 4500
 $Comp
-L BusSimulator-rescue:GNDREF #PWR0107
+L Carrier-Board-rescue:GNDREF-BusSimulator-rescue #PWR0107
 U 1 1 5BC5364F
 P 7300 4800
@@
 $EndComp
 $Comp
-L BusSimulator-rescue:GNDREF #PWR0108
+L Carrier-Board-rescue:GNDREF-BusSimulator-rescue #PWR0108
 U 1 1 5BC5377A
 P 8100 5300
@@
 	6900 5500 7100 5500
 $Comp
-L BusSimulator-rescue:GNDREF #PWR0109
+L Carrier-Board-rescue:GNDREF-BusSimulator-rescue #PWR0109
 U 1 1 5BCD9D55
 P 6300 5800
@@
 	6300 3700 6300 3900
 $Comp
-L BusSimulator-rescue:GNDREF #PWR0110
+L Carrier-Board-rescue:GNDREF-BusSimulator-rescue #PWR0110
 U 1 1 5BD25D30
 P 4950 4050
@@
 NoConn ~ 6900 5400
 $Comp
-L BusSimulator-rescue:R R14
+L Carrier-Board-rescue:R-BusSimulator-rescue R14
 U 1 1 5BD56E81
 P 6200 9550
@@
 	5900 9550 6050 9550
 $Comp
-L BusSimulator-rescue:GNDREF #PWR0111
+L Carrier-Board-rescue:GNDREF-BusSimulator-rescue #PWR0111
 U 1 1 5BDA5099
 P 6050 6150
